File: cad/robo_car.kicad_pcb (KiCad board)
At the start: 2 copper layers, 100 x 100 mm, 77 parts, among them J1 Conn_01x06_MountingPin, J16 Conn_01x02_MountingPin, J2 ftdi_conn, J3 Conn_01x06_MountingPin, J4 Conn_01x04, J5 Conn_01x04, J6 Conn_01x06_MountingPin, J8 Conn_01x02_MountingPin, SW1 SW_Push, SW2 SW_Push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

Commit message: Traces started, chicken cooking
Parts:
- added H21: MountingHole, MountingHole:MountingHole_2.7mm_M2.5_ISO14580, F.Cu at (111.9, 119.6)
- added H22: MountingHole, MountingHole:MountingHole_2.7mm_M2.5_ISO14580, F.Cu at (191.9, 119.6)
- added H23: MountingHole, MountingHole:MountingHole_2.7mm_M2.5_ISO14580, F.Cu at (191.9, 137.6)
- added H24: MountingHole, MountingHole:MountingHole_2.7mm_M2.5_ISO14580, F.Cu at (111.9, 137.6)
- moved H15 141.3 mm to (196.9, 103.6)
- moved H14 127.5 mm to (106.9, 148.6)
- moved H20 124.1 mm to (196.9, 93.6)
- moved H3 109.0 mm to (176.9, 78.6)
- moved H18 107.0 mm to (196.9, 83.6)
- moved H13 98.5 mm to (71.9, 73.6)
- moved H2 84.8 mm to (166.9, 58.6)
- moved H17 75.6 mm to (106.9, 103.6)
- moved H16 67.8 mm to (146.9, 58.6)
- moved H10 63.3 mm to (156.9, 58.6)
- moved H5 62.3 mm to (106.9, 93.6)
- moved H19 60.4 mm to (196.9, 148.6)
- moved H11 55.4 mm to (124.9, 78.6)
- moved H8 52.8 mm to (136.9, 58.6)
- moved H12 47.8 mm to (106.9, 83.6)
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Routing:
- net +3V3: track 41.7 -> 177.3 mm
- net /VREG_OUT: track 0.00 -> 117.1 mm
- net VBUS: track 0.00 -> 93.9 mm, vias 0 -> 2
- net /RESET: track 0.00 -> 34.7 mm, vias 0 -> 2
- net /BOOT: track 0.00 -> 16.9 mm, vias 0 -> 2
- net /MOTOR_R_2: track 0.00 -> 9.96 mm
- net Net-(D1-Pad1): track 0.00 -> 9.85 mm
- net /MOTOR_R_1: track 0.00 -> 7.55 mm
- net /MOTOR_L_2: track 0.00 -> 5.72 mm
- net /RXD0: track 0.00 -> 4.79 mm
- net /TXDO: track 0.00 -> 4.67 mm
- net /MOTOR_L_1: track 0.00 -> 3.95 mm
- net Net-(D13-Pad1): track 0.00 -> 2.01 mm
- net Net-(D12-Pad1): track 0.00 -> 2.01 mm
- net Net-(D14-Pad1): track 0.00 -> 2.01 mm
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- added copper zone on B.Cu, net GND
- added copper zone on F.Cu, net Net-(D1-Pad1)
Other:
- outline, holes or cut-outs redrawn
- board text added: "^ Reset :)"

Commit message: Handy highway comes in from the other left *beep beep*
Parts:
- added H25: MountingHole, MountingHole:MountingHole_3.2mm_M3_ISO14580, F.Cu at (196.9, 78.6)
- added J7: Conn_01x02_MountingPin, Connector_JST:JST_XH_2_VERTICAL, F.Cu at (190.9, 96.8)
- H1, H10, H11, H12, H13, H14, H15, H16, H17, H18, H19, H2, H20, H3, H4, H5, H6, H7, H8, H9: footprint MountingHole:MountingHole_3.2mm_M3_ISO14580_Pad -> MountingHole:MountingHole_3.2mm_M3_ISO14580
- moved H13 35.4 mm to (106.9, 78.6)
- moved J1 21.1 mm to (184.3, 80.0), turned to 180 degrees
- moved J6 20.0 mm to (120.0, 79.6), turned to 180 degrees
- moved H11 8.58 mm to (131.9, 73.6)
- moved H3 7.07 mm to (171.9, 73.6)
- moved H12 5.00 mm to (106.9, 88.6)
- moved H15 5.00 mm to (196.9, 108.6)
- moved H17 5.00 mm to (106.9, 108.6)
- moved H18 5.00 mm to (196.9, 88.6)
- moved H20 5.00 mm to (196.9, 98.6)
- moved H5 5.00 mm to (106.9, 98.6)
- moved D6 3.54 mm to (182.2, 111.7)
- moved R5 3.54 mm to (186.9, 106.8)
- moved C10 3.54 mm to (182.3, 106.2)
- moved D3 3.54 mm to (186.9, 110.8)
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Connections:
- J1 pad 1: /ANALOG_C -> /ANALOG_A
- J1 pad 2: /ANALOG_A -> /ANALOG_B
- J1 pad 3: /ANALOG_B -> /ANALOG_C
- J16 pad 1: Net-(J16-Pad1) -> Net-(U4-Pad7)
- J16 pad 2: Net-(J16-Pad2) -> Net-(U4-Pad8)
- U3 pad 11: /SERVO_0 -> /MOTOR_L_2
- U3 pad 12: /SERVO_1 -> /HBT_LED
- U3 pad 13: /INPUT_C -> /MOTOR_L_1
- U3 pad 14: /SDA -> /NEO_STATUS
- U3 pad 16: /MOTOR_L_1 -> unconnected-(U3-Pad16)
- U3 pad 28: /NEO_STATUS -> /SDA
- U3 pad 29: /HBT_LED -> unconnected-(U3-Pad29)
- U3 pad 30: /MOTOR_L_2 -> unconnected-(U3-Pad30)
- U3 pad 6: /ANALOG_C -> /ANALOG_B
- U3 pad 7: /ANALOG_B -> /ANALOG_C
- U4 pad 7: Net-(J16-Pad2) -> Net-(U4-Pad7)
- U4 pad 8: Net-(J16-Pad1) -> Net-(U4-Pad8)
Routing:
- net /ANALOG_A: track 0.00 -> 74.6 mm
- net /ANALOG_B: track 0.00 -> 73.0 mm
- net /ANALOG_C: track 0.00 -> 71.4 mm
- net /ANALOG_D: track 0.00 -> 69.6 mm
- net /FUNCTION_BUTTON: track 0.00 -> 48.9 mm, vias 0 -> 2
- net /NEO_STATUS: track 0.00 -> 42.8 mm, vias 0 -> 4
- net /HBT_LED: track 0.00 -> 38.8 mm, vias 0 -> 4
- net /MOTOR_L_1: track 3.95 -> 35.2 mm, vias 0 -> 2
- net /MOTOR_L_2: track 5.72 -> 36.1 mm
- net /MOTOR_R_2: track 9.96 -> 40.2 mm
- net /MOTOR_R_1: track 7.55 -> 37.6 mm
- net Net-(U4-Pad7): track 0.00 -> 22.6 mm
- net Net-(U4-Pad8): track 0.00 -> 21.9 mm
- net /VREG_OUT: track 117.1 -> 133.8 mm, vias 0 -> 2
- net Net-(J8-Pad2): track 0.00 -> 15.9 mm
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Other:
- board text added: "0"

Commit message: Noise complaint, V cops on the way
Parts:
- moved J8 5.72 mm to (129.6, 113.4)
- moved D12 4.95 mm to (158.0, 123.7)
- moved R4 4.95 mm to (158.0, 127.3)
- moved R9 4.95 mm to (162.0, 127.3)
- moved D13 4.95 mm to (160.1, 123.7)
- moved D15 4.95 mm to (164.2, 123.7)
- moved D14 4.95 mm to (162.1, 123.7)
- moved R10 4.95 mm to (164.3, 127.2)
- moved R8 4.95 mm to (159.9, 127.3)
- moved C9 3.98 mm to (135.4, 138.6)
- moved C15 3.84 mm to (135.3, 140.5)
- moved U5 3.63 mm to (135.5, 133.3)
- moved J5 3.61 mm to (130.3, 147.5)
- moved J2 3.15 mm to (141.7, 147.4)
- moved C1 2.50 mm to (116.7, 147.2)
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Connections:
- J4 pad 1: /CAN_L -> /CAN_H
- J4 pad 2: /CAN_H -> /CAN_L
- J5 pad 1: /CAN_L -> /CAN_H
- J5 pad 2: /CAN_H -> /CAN_L
- U3 pad 16: unconnected-(U3-Pad16) -> /INPUT_D
- U3 pad 28: /SDA -> /INPUT_C
- U3 pad 29: unconnected-(U3-Pad29) -> /INPUT_A
- U3 pad 30: unconnected-(U3-Pad30) -> /INPUT_B
- U3 pad 31: /SCL -> /SERVO_1
- U3 pad 33: /INPUT_A -> /SERVO_0
- U3 pad 36: /INPUT_B -> /SCL
- U3 pad 37: /INPUT_D -> /SDA
Routing:
- net /INPUT_D: track 0.00 -> 92.0 mm, vias 0 -> 4
- net /INPUT_B: track 0.00 -> 91.5 mm, vias 0 -> 2
- net /INPUT_A: track 0.00 -> 90.3 mm, vias 0 -> 2
- net /SDA: track 0.00 -> 89.2 mm, vias 0 -> 2
- net /INPUT_C: track 0.00 -> 89.0 mm, vias 0 -> 2
- net /SCL: track 0.00 -> 85.1 mm, vias 0 -> 2
- net /SERVO_0: track 0.00 -> 77.4 mm
- net /SERVO_1: track 0.00 -> 75.0 mm
- net +3V3: track 175.2 -> 241.1 mm
- net /NEO_BAR: track 0.00 -> 62.7 mm, vias 0 -> 2
- net /CAN_H: track 0.00 -> 33.7 mm, vias 0 -> 2
- net /CAN_L: track 0.00 -> 31.1 mm
- net /CAN_SLP: track 0.00 -> 22.9 mm, vias 0 -> 2
- net /CAN_TX: track 0.00 -> 18.3 mm, vias 0 -> 2
- net /CAN_RX: track 0.00 -> 13.5 mm, vias 0 -> 2
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Other:
- outline, holes or cut-outs redrawn
- board text added: "3"
- board text added: "G"

Commit message: Roger, rodger? Wait it's Ralphie!
Routing:
- net /VREG_OUT: track 134.0 -> 134.8 mm
- net Net-(J8-Pad1): vias 2 -> 3
- net GND: vias 106 -> 276
Other:
- board text added: "1"
- board text added: "12"
- board text added: "13"
- board text added: "17"
- board text added: "18"
- board text added: "19"
- board text added: "2"
- board text added: "21"
- board text added: "22"
- board text added: "23"
- board text added: "27"
- board text added: "32"
- board text added: "34"
- board text added: "35"
- board text added: "36"
- board text added: "39"
- board text added: "3V"
- board text added: "4"
- board text added: "5"
- board text added: "5V"
- board text added: "Button"
- board text added: "Function"
- board text added: "Louie"
- board text added: "Made by Olivia & Andrew 2022"
- board text added: "Ralphie"

Commit message: Dapper drawings, forward and behindward!
Parts:
- added G***: LOGO, Drawing:mustache, F.Cu at (151.5, 104.0)
- added G***: LOGO, Drawing:backside, B.Cu at (152.5, 104.5)

Commit message: Olivia Attempts Andrewism, and Abolishes Her Awesome Highway
Parts:
- added H26: MountingHole, MountingHole:MountingHole_3.2mm_M3_ISO14580, F.Cu at (170.0, 77.0)
- added H27: MountingHole, MountingHole:MountingHole_3.2mm_M3_ISO14580, F.Cu at (130.0, 77.0)
- moved C1 19.4 mm to (113.8, 128.0)
- moved D7 12.4 mm to (125.6, 132.0), turned to 180 degrees
- moved J8 9.62 mm to (136.8, 107.0)
- moved C15 9.23 mm to (139.0, 132.0), turned to -90 degrees
- moved H1 8.83 mm to (130.0, 115.0)
- moved H11 8.83 mm to (130.0, 65.0)
- moved H12 8.83 mm to (105.0, 80.0)
- moved H13 8.83 mm to (105.0, 70.0)
- moved H15 8.83 mm to (195.0, 100.0)
- moved H17 8.83 mm to (105.0, 100.0)
- moved H18 8.83 mm to (195.0, 80.0)
- moved H20 8.83 mm to (195.0, 90.0)
- moved H25 8.83 mm to (195.0, 70.0)
- moved H3 8.83 mm to (170.0, 65.0)
- moved H5 8.83 mm to (105.0, 90.0)
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Connections:
- U3 pad 13: /MOTOR_L_1 -> /NEO_STATUS
- U3 pad 14: /NEO_STATUS -> /MOTOR_L_1
Routing:
- net /INPUT_D: track 92.0 -> 0.00 mm, vias 4 -> 0
- net /INPUT_B: track 91.5 -> 0.00 mm, vias 2 -> 0
- net /INPUT_A: track 90.3 -> 0.00 mm, vias 2 -> 0
- net /SDA: track 89.2 -> 0.00 mm, vias 2 -> 0
- net /INPUT_C: track 89.0 -> 0.00 mm, vias 2 -> 0
- net /SCL: track 85.1 -> 0.00 mm, vias 2 -> 0
- net /SERVO_0: track 77.4 -> 0.00 mm
- net /SERVO_1: track 75.0 -> 0.00 mm
- net /NEO_BAR: track 62.7 -> 0.00 mm, vias 2 -> 0
- net /VREG_OUT: track 134.8 -> 81.6 mm, vias 4 -> 2
- net +3V3: track 241.1 -> 193.2 mm, vias 2 -> 0
- net /FUNCTION_BUTTON: track 50.4 -> 4.23 mm, vias 2 -> 0
- net /NEO_STATUS: track 42.8 -> 0.00 mm, vias 4 -> 0
- net /HBT_LED: track 38.8 -> 0.00 mm, vias 4 -> 0
- net /MOTOR_L_1: track 38.9 -> 2.61 mm, vias 2 -> 0
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- added copper zone on F.Cu, net /VREG_OUT
- added copper zone on B.Cu, net VBUS
- added copper zone on F.Cu, net VBUS
Other:
- outline, holes or cut-outs redrawn
- board text removed: "Ralphie"

Commit message: Andrew Puts a Traffic Cone on Olivia's Happy Highway
Parts:
- added C16: 47uF, Capacitor_SMD:CP_Elec_6.3x7.7, F.Cu at (200.2, 115.0)
Changed lines of the file:
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@@
     )
   )
+  (footprint "Capacitor_SMD:CP_Elec_6.3x7.7" (layer "F.Cu")
+    (at 200.2 115)
+    (descr "SMD capacitor, aluminum electrolytic, Nichicon, 6.3x7.7mm")
+    (tags "capacitor electrolytic")
+    (property "Sheetfile" "robo_car.kicad_sch")
+    (property "Sheetname" "")
+    (attr smd)
+    (fp_text reference "C16" (at 0 -4.35) (layer "F.SilkS")
+      (effects (font (size 1 1) (thickness 0.15)))
+    )
+    (fp_text value "47uF" (at 0 4.35) (layer "F.Fab")
+      (effects (font (size 1 1) (thickness 0.15)))
+    )
+    (fp_text user "${REFERENCE}" (at 0 0) (layer "F.Fab")
+      (effects (font (size 1 1) (thickness 0.15)))
+    )
+    (fp_line (start 3.41 -3.41) (end 3.41 -1.06) (layer "F.SilkS") (width 0.12))
+    (fp_line (start -4.04375 -2.24125) (end -4.04375 -1.45375) (layer "F.SilkS") (width 0.12))
+    (fp_line (start -3.41 2.345563) (end -2.345563 3.41) (layer "F.SilkS") (width 0.12))
+    (fp_line (start -3.41 -2.345563) (end -3.41 -1.06) (layer "F.SilkS") (width 0.12))
+    (fp_line (start -4.4375 -1.8475) (end -3.65 -1.8475) (layer "F.SilkS") (width 0.12))
+    (fp_line (start -2.345563 3.41) (end 3.41 3.41) (layer "F.SilkS") (width 0.12))
+    (fp_line (start -3.41 2.345563) (end -3.41 1.06) (layer "F.SilkS") (width 0.12))
+    (fp_line (start 3.41 3.41) (end 3.41 1.06) (layer "F.SilkS") (width 0.12))
+    (fp_line (start -2.345563 -3.41) (end 3.41 -3.41) (layer "F.SilkS") (width 0.12))
+    (fp_line (start -3.41 -2.345563) (end -2.345563 -3.41) (layer "F.SilkS") (width 0.12))
+    (fp_line (start -4.7 -1.05) (end -4.7 1.05) (layer "F.CrtYd") (width 0.05))
+    (fp_line (start -4.7 1.05) (end -3.55 1.05) (layer "F.CrtYd") (width 0.05))
+    (fp_line (start -3.55 1.05) (end -3.55 2.4) (layer "F.CrtYd") (width 0.05))
+    (fp_line (start 4.7 -1.05) (end 4.7 1.05) (layer "F.CrtYd") (width 0.05))
+    (fp_line (start 3.55 -1.05) (end 4.7 -1.05) (layer "F.CrtYd") (width 0.05))
+    (fp_line (start -3.55 -1.05) (end -4.7 -1.05) (layer "F.CrtYd") (width 0.05))
+    (fp_line (start 3.55 -3.55) (end 3.55 -1.05) (layer "F.CrtYd") (width 0.05))
+    (fp_line (start 4.7 1.05) (end 3.55 1.05) (layer "F.CrtYd") (width 0.05))
+    (fp_line (start -2.4 -3.55) (end 3.55 -3.55) (layer "F.CrtYd") (width 0.05))
+    (fp_line (start -3.55 -2.4) (end -3.55 -1.05) (layer "F.CrtYd") (width 0.05))
+    (fp_line (start -2.4 3.55) (end 3.55 3.55) (layer "F.CrtYd") (width 0.05))
+    (fp_line (start 3.55 1.05) (end 3.55 3.55) (layer "F.CrtYd") (width 0.05))
+    (fp_line (start -3.55 -2.4) (end -2.4 -3.55) (layer "F.CrtYd") (width 0.05))
+    (fp_line (start -3.55 2.4) (end -2.4 3.55) (layer "F.CrtYd") (width 0.05))
+    (fp_line (start -3.3 -2.3) (end -3.3 2.3) (layer "F.Fab") (width 0.1))
+    (fp_line (start -2.3 -3.3) (end 3.3 -3.3) (layer "F.Fab") (width 0.1))
+    (fp_line (start -2.704838 -1.33) (end -2.074838 -1.33) (layer "F.Fab") (width 0.1))
+    (fp_line (start -3.3 2.3) (end -2.3 3.3) (layer "F.Fab") (width 0.1))
+    (fp_line (start -2.3 3.3) (end 3.3 3.3) (layer "F.Fab") (width 0.1))
+    (fp_line (start 3.3 -3.3) (end 3.3 3.3) (layer "F.Fab") (width 0.1))
+    (fp_line (start -3.3 -2.3) (end -2.3 -3.3) (layer "F.Fab") (width 0.1))
+    (fp_line (start -2.389838 -1.645) (end -2.389838 -1.015) (layer "F.Fab") (width 0.1))
+    (fp_circle (center 0 0) (end 3.15 0) (layer "F.Fab") (width 0.1) (fill none))
+    (pad "1" smd roundrect locked (at -2.7 0) (size 3.5 1.6) (layers "F.Cu" "F.Paste" "F.Mask") (roundrect_rratio 0.15625)
+      (net 15 "VBUS") (pintype "passive"))
+    (pad "2" smd roundrect locked (at 2.7 0) (size 3.5 1.6) (layers "F.Cu" "F.Paste" "F.Mask") (roundrect_rratio 0.15625)
+      (net 4 "GND") (pintype "passive"))
+    (model "${KICAD6_3DMODEL_DIR}/Capacitor_SMD.3dshapes/CP_Elec_6.3x7.7.wrl"
+      (offset (xyz 0 0 0))
+      (scale (xyz 1 1 1))
+      (rotate (xyz 0 0 0))
+    )
+  )
   (footprint "Resistor_SMD:R_0603_1608Metric" (layer "F.Cu")
     (at 185.04 103.2275 -90)
@@
       (net 13 "/HBT_LED") (pinfunction "A2-IO27") (pintype "bidirectional"))
     (pad "13" smd rect (at -8.5 6.985 180) (size 2 0.9) (layers "F.Cu" "F.Paste" "F.Mask")
-      (net 10 "/NEO_STATUS") (pinfunction "HSCK-A2-IO14") (pintype "bidirectional"))
+      (net 10 "/NEO_STATUS") (pinfunction "NOISE@BOOT-HSCK-A2-IO14") (pintype "bidirectional"))
     (pad "14" smd rect (at -8.5 8.255 180) (size 2 0.9) (layers "F.Cu" "F.Paste" "F.Mask")
-      (net 55 "/MOTOR_L_1") (pinfunction "HMISO-A2-IO12") (pintype "bidirectional"))
+      (net 55 "/MOTOR_L_1") (pinfunction "LOW@BOOT-HMISO-A2-IO12") (pintype "bidirectional"))
     (pad "15" smd rect (at -5.715 9.255 90) (size 2 0.9) (layers "F.Cu" "F.Paste" "F.Mask")
       (net 4 "GND") (pinfunction "GND") (pintype "passive"))
@@
       (net 42 "unconnected-(U3-Pad22)") (pinfunction "SDI/SD1") (pintype "bidirectional+no_connect"))
     (pad "23" smd rect (at 4.445 9.255 270) (size 2 0.9) (layers "F.Cu" "F.Paste" "F.Mask")
-      (net 16 "/NEO_BAR") (pinfunction "A2-IO15") (pintype "bidirectional"))
+      (net 16 "/NEO_BAR") (pinfunction "NOISE@BOOT-A2-IO15") (pintype "bidirectional"))
     (pad "24" smd rect (at 5.715 9.255 270) (size 2 0.9) (layers "F.Cu" "F.Paste" "F.Mask")
-      (net 43 "/CAN_SLP") (pinfunction "A2-IO2") (pintype "bidirectional"))
+      (net 43 "/CAN_SLP") (pinfunction "LOW@BOOT-A2-IO2") (pintype "bidirectional"))
     (pad "25" smd rect (at 8.5 8.255 180) (size 2 0.9) (layers "F.Cu" "F.Paste" "F.Mask")
       (net 21 "/BOOT") (pinfunction "BOOT-A2-IO0") (pintype "bidirectional"))

Commit message: Sleepy Olivia Draws Lines
Parts:
- moved C14 2.51 mm to (137.6, 79.9)
- moved C22 2.51 mm to (164.6, 79.7)
- moved C18 2.51 mm to (151.0, 79.9)
- moved C21 2.51 mm to (157.4, 79.9)
- moved C8 2.51 mm to (144.3, 79.9)
- moved D10 2.51 mm to (158.8, 84.6)
- moved D11 2.51 mm to (165.6, 84.6)
- moved D4 2.51 mm to (138.6, 84.6)
- moved D5 2.51 mm to (145.3, 84.6)
- moved D9 2.51 mm to (152.1, 84.6)
- moved SW1 2.28 mm to (188.0, 103.2)
- moved R3 2.19 mm to (189.8, 108.7), turned to -90 degrees
- moved J7 1.81 mm to (188.9, 91.3)
- moved J8 1.50 mm to (136.0, 105.7)
- moved J16 1.26 mm to (166.8, 106.3)
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Routing:
- net /INPUT_B: track 0.00 -> 108.8 mm
- net /NEO_BAR: track 0.00 -> 107.2 mm
- net /INPUT_A: track 0.00 -> 105.7 mm
- net /INPUT_C: track 0.00 -> 102.6 mm
- net /SDA: track 0.00 -> 84.4 mm
- net /SCL: track 0.00 -> 83.1 mm
- net /SERVO_0: track 0.00 -> 78.6 mm
- net /SERVO_1: track 0.00 -> 75.6 mm
- net /FUNCTION_BUTTON: track 4.23 -> 49.7 mm, vias 0 -> 2
- net /CAN_SLP: track 2.96 -> 33.2 mm, vias 2 -> 4
- net +3V3: track 193.2 -> 216.5 mm, vias 0 -> 2
- net /BOOT: track 21.9 -> 0.00 mm, vias 2 -> 0
- net VBUS: track 69.9 -> 51.3 mm
- net Net-(J8-Pad1): track 14.9 -> 18.7 mm
- net Net-(D8-Pad1): track 0.00 -> 3.03 mm
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