File: cad/robo_car.kicad_sch (KiCad schematic)
At the start: 77 parts, among them J1 Conn_01x06_MountingPin, J16 Conn_01x02_MountingPin, J2 ftdi_conn, J3 Conn_01x06_MountingPin, J4 Conn_01x04, J5 Conn_01x04, J6 Conn_01x06_MountingPin, J8 Conn_01x02_MountingPin, SW1 SW_Push, SW2 SW_Push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

Commit message: Traces started, chicken cooking
Parts:
- added H21, H22, H23, H24: MountingHole, MountingHole:MountingHole_2.7mm_M2.5_ISO14580, symbol Mechanical:MountingHole
Changed lines of the file:
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@@
+    )
+  )
+  (symbol (lib_id "Mechanical:MountingHole") (at 187.96 147.32 0) (unit 1)
+    (in_bom yes) (on_board yes) (fields_autoplaced)
+    (property "Reference" "H22" (id 0) (at 190.5 146.4115 0)
+      (effects (font (size 1.27 1.27)) (justify left))
+    )
+    (property "Value" "MountingHole" (id 1) (at 190.5 149.1866 0)
+      (effects (font (size 1.27 1.27)) (justify left))
+    )
+    (property "Footprint" "MountingHole:MountingHole_2.7mm_M2.5_ISO14580" (id 2) (at 187.96 147.32 0)
+      (effects (font (size 1.27 1.27)) hide)
+    )
+    (property "Datasheet" "~" (id 3) (at 187.96 147.32 0)
+      (effects (font (size 1.27 1.27)) hide)
     )
   )
@@
     )
   )
+  (symbol (lib_id "Mechanical:MountingHole") (at 187.96 132.715 0) (unit 1)
+    (in_bom yes) (on_board yes) (fields_autoplaced)
+    (property "Reference" "H21" (id 0) (at 190.5 131.8065 0)
+      (effects (font (size 1.27 1.27)) (justify left))
+    )
+    (property "Value" "MountingHole" (id 1) (at 190.5 134.5816 0)
+      (effects (font (size 1.27 1.27)) (justify left))
+    )
+    (property "Footprint" "MountingHole:MountingHole_2.7mm_M2.5_ISO14580" (id 2) (at 187.96 132.715 0)
+      (effects (font (size 1.27 1.27)) hide)
+    )
+    (property "Datasheet" "~" (id 3) (at 187.96 132.715 0)
+      (effects (font (size 1.27 1.27)) hide)
+    )
+  )
   (symbol (lib_id "power:GND") (at 74.295 34.925 0) (mirror y) (unit 1)
     (in_bom yes) (on_board yes)
@@
     )
     (pin "1")
+  )
+  (symbol (lib_id "Mechanical:MountingHole") (at 189.865 160.02 0) (unit 1)
+    (in_bom yes) (on_board yes) (fields_autoplaced)
+    (property "Reference" "H24" (id 0) (at 192.405 159.1115 0)
+      (effects (font (size 1.27 1.27)) (justify left))
+    )
+    (property "Value" "MountingHole" (id 1) (at 192.405 161.8866 0)
+      (effects (font (size 1.27 1.27)) (justify left))
+    )
+    (property "Footprint" "MountingHole:MountingHole_2.7mm_M2.5_ISO14580" (id 2) (at 189.865 160.02 0)
+      (effects (font (size 1.27 1.27)) hide)
+    )
+    (property "Datasheet" "~" (id 3) (at 189.865 160.02 0)
+      (effects (font (size 1.27 1.27)) hide)
+    )
   )
   (symbol (lib_id "power:GND") (at 86.36 237.49 0) (mirror y) (unit 1)
@@
     (pin "2")
   )
+  (symbol (lib_id "Mechanical:MountingHole") (at 188.595 140.335 0) (unit 1)
+    (in_bom yes) (on_board yes) (fields_autoplaced)
+    (property "Reference" "H23" (id 0) (at 191.135 139.4265 0)
+      (effects (font (size 1.27 1.27)) (justify left))
+    )
+    (property "Value" "MountingHole" (id 1) (at 191.135 142.2016 0)
+      (effects (font (size 1.27 1.27)) (justify left))
+    )
+    (property "Footprint" "MountingHole:MountingHole_2.7mm_M2.5_ISO14580" (id 2) (at 188.595 140.335 0)
+      (effects (font (size 1.27 1.27)) hide)
+    )
+    (property "Datasheet" "~" (id 3) (at 188.595 140.335 0)
+      (effects (font (size 1.27 1.27)) hide)
+    )
+  )
   (symbol (lib_id "Mechanical:MountingHole") (at 135.89 74.93 0) (unit 1)
     (in_bom yes) (on_board yes) (fields_autoplaced)
@@
       (reference "H20") (unit 1) (value "MountingHole") (footprint "MountingHole:MountingHole_3.2mm_M3_ISO14580_Pad")
     )
+    (path "/8e417d1c-3cb9-46fd-ba99-6ef1379483b6"
+      (reference "H21") (unit 1) (value "MountingHole") (footprint "MountingHole:MountingHole_2.7mm_M2.5_ISO14580")
+    )
+    (path "/2cdad8ef-b5c8-42b4-91da-9d5f6d9b006b"
+      (reference "H22") (unit 1) (value "MountingHole") (footprint "MountingHole:MountingHole_2.7mm_M2.5_ISO14580")
+    )
+    (path "/d49dbff2-b983-4798-8ccf-c45ba353b537"
+      (reference "H23") (unit 1) (value "MountingHole") (footprint "MountingHole:MountingHole_2.7mm_M2.5_ISO14580")
+    )
+    (path "/972e61ff-fa80-472d-a039-f69ba260725a"
+      (reference "H24") (unit 1) (value "MountingHole") (footprint "MountingHole:MountingHole_2.7mm_M2.5_ISO14580")
+    )
     (path "/ba845734-cb29-4a35-9ff6-e58ec1810bec"

Commit message: Handy highway comes in from the other left *beep beep*
Parts:
- added H25: MountingHole, MountingHole:MountingHole_3.2mm_M3_ISO14580, symbol Mechanical:MountingHole
- added J7: Conn_01x02_MountingPin, Connector_JST:JST_XH_2_VERTICAL, symbol Connector_Generic_MountingPin:Conn_01x02_MountingPin
- H1, H10, H11, H12, H13, H14, H15, H16, H17, H18, H19, H2, H20, H3, H4, H5, H6, H7, H8, H9: footprint MountingHole:MountingHole_3.2mm_M3_ISO14580_Pad -> MountingHole:MountingHole_3.2mm_M3_ISO14580
Connections:
- net ANALOG_A: now also J1.1 (Pin_1); no longer J1.2 (Pin_2)
- net ANALOG_B: now also J1.2 (Pin_2), U3.6 (inputOnly-noPU-A1-IO34); no longer J1.3 (Pin_3), U3.7 (inputOnly-noPU-A1-IO35)
- net ANALOG_C: now also J1.3 (Pin_3), U3.7 (inputOnly-noPU-A1-IO35); no longer J1.1 (Pin_1), U3.6 (inputOnly-noPU-A1-IO34)
- net GND: now also J7.2 (Pin_2), J7.MP (MountPin)
- net HBT_LED: now also U3.12 (A2-IO27); no longer U3.29 (IO5)
- net INPUT_C: no longer U3.13 (HSCK-A2-IO14)
- net MOTOR_L_1: now also U3.13 (HSCK-A2-IO14); no longer U3.16 (HMOSI-A2-IO13)
- net MOTOR_L_2: now also U3.11 (SDA1-DAC2-A2-IO26); no longer U3.30 (SCL0-VCLK-IO18)
- net NEO_STATUS: now also U3.14 (HMISO-A2-IO12); no longer U3.28 (IO17)
- net SDA: now also U3.28 (IO17); no longer U3.14 (HMISO-A2-IO12)
- net SERVO_0: no longer U3.11 (SDA1-DAC2-A2-IO26)
- net SERVO_1: no longer U3.12 (A2-IO27)
- net VREG_OUT: now also J7.1 (Pin_1)
- net at U4.7 (OUT4): now also J16.1 (Pin_1); no longer J16.2 (Pin_2)
- net at U4.8 (OUT3): now also J16.2 (Pin_2); no longer J16.1 (Pin_1)
Other:
- note added: "*"
- moved on the sheet: J16

Commit message: Noise complaint, V cops on the way
Connections:
- net CAN_H: now also J4.1 (Pin_1), J5.1 (Pin_1); no longer J4.2 (Pin_2), J5.2 (Pin_2)
- net CAN_L: now also J4.2 (Pin_2), J5.2 (Pin_2); no longer J4.1 (Pin_1), J5.1 (Pin_1)
- net INPUT_A: now also U3.29 (IO5); no longer U3.33 (IO21)
- net INPUT_B: now also U3.30 (SCL0-VCLK-IO18); no longer U3.36 (IO22)
- net INPUT_C: now also U3.28 (IO17)
- net INPUT_D: now also U3.16 (HMOSI-A2-IO13); no longer U3.37 (VMOSI-IO23)
- net SCL: now also U3.36 (IO22); no longer U3.31 (SDA0-VMISO-IO19)
- net SDA: now also U3.37 (VMOSI-IO23); no longer U3.28 (IO17)
- net SERVO_0: now also U3.33 (IO21)
- net SERVO_1: now also U3.31 (SDA0-VMISO-IO19)
Changed lines of the file:
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@@
     (effects (font (size 1.27 1.27)) (justify left bottom))
   )
-  (label "SDA" (at 316.23 170.18 180)
+  (label "SDA" (at 314.96 182.88 180)
     (effects (font (size 1.27 1.27)) (justify right bottom))
   )
-  (label "CAN_H" (at 394.97 130.81 90)
+  (label "CAN_H" (at 392.43 130.81 90)
     (effects (font (size 1.27 1.27)) (justify left bottom))
   )
@@
     (effects (font (size 1.27 1.27)) (justify right bottom))
   )
-  (label "CAN_L" (at 392.43 130.81 90)
+  (label "CAN_L" (at 394.97 130.81 90)
     (effects (font (size 1.27 1.27)) (justify left bottom))
   )
@@
     (effects (font (size 1.27 1.27)) (justify right bottom))
   )
-  (label "INPUT_C" (at 320.675 142.24 180)
+  (label "INPUT_C" (at 316.23 170.18 180)
     (effects (font (size 1.27 1.27)) (justify right bottom))
   )
@@
     (effects (font (size 1.27 1.27)) (justify left bottom))
   )
-  (label "SERVO_0" (at 321.945 147.955 180)
+  (label "SERVO_0" (at 314.96 177.8 180)
     (effects (font (size 1.27 1.27)) (justify right bottom))
   )
@@
     (effects (font (size 1.27 1.27)) (justify right bottom))
   )
-  (label "CAN_H" (at 394.97 152.4 90)
+  (label "CAN_H" (at 392.43 152.4 90)
     (effects (font (size 1.27 1.27)) (justify left bottom))
   )
@@
     (effects (font (size 1.27 1.27)) (justify left bottom))
   )
-  (label "INPUT_B" (at 314.96 180.34 180)
+  (label "INPUT_B" (at 314.96 172.72 180)
     (effects (font (size 1.27 1.27)) (justify right bottom))
   )
@@
     (effects (font (size 1.27 1.27)) (justify right bottom))
   )
-  (label "INPUT_D" (at 314.96 182.88 180)
+  (label "INPUT_D" (at 314.96 160.02 180)
     (effects (font (size 1.27 1.27)) (justify right bottom))
   )
@@
     (effects (font (size 1.27 1.27)) (justify left bottom))
   )
-  (label "INPUT_A" (at 314.96 177.8 180)
+  (label "INPUT_A" (at 312.42 154.94 180)
     (effects (font (size 1.27 1.27)) (justify right bottom))
   )
@@
     (effects (font (size 1.27 1.27)) (justify left bottom))
   )
-  (label "SCL" (at 314.96 175.26 180)
+  (label "SCL" (at 314.96 180.34 180)
     (effects (font (size 1.27 1.27)) (justify right bottom))
   )
@@
     (effects (font (size 1.27 1.27)) (justify right bottom))
   )
-  (label "SERVO_1" (at 321.437 151.511 180)
+  (label "SERVO_1" (at 314.96 175.26 180)
     (effects (font (size 1.27 1.27)) (justify right bottom))
   )
@@
     (effects (font (size 1.27 1.27)) (justify left bottom))
   )
-  (label "CAN_L" (at 392.43 152.4 90)
+  (label "CAN_L" (at 394.97 152.4 90)
     (effects (font (size 1.27 1.27)) (justify left bottom))
   )

Commit message: Olivia Attempts Andrewism, and Abolishes Her Awesome Highway
Parts:
- added H26, H27: MountingHole, MountingHole:MountingHole_3.2mm_M3_ISO14580, symbol Mechanical:MountingHole
Connections:
- net MOTOR_L_1: now also U3.14 (HMISO-A2-IO12); no longer U3.13 (HSCK-A2-IO14)
- net NEO_STATUS: now also U3.13 (HSCK-A2-IO14); no longer U3.14 (HMISO-A2-IO12)
Changed lines of the file:
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@@
     (effects (font (size 1.27 1.27)) (justify left bottom))
   )
-  (label "MOTOR_L_1" (at 314.96 162.56 180)
+  (label "MOTOR_L_1" (at 314.96 157.48 180)
     (effects (font (size 1.27 1.27)) (justify right bottom))
   )
@@
     (effects (font (size 1.27 1.27)) (justify left bottom))
   )
-  (label "NEO_STATUS" (at 314.96 157.48 180)
+  (label "NEO_STATUS" (at 314.96 162.56 180)
     (effects (font (size 1.27 1.27)) (justify right bottom))
   )
@@
     (pin "2")
   )
+  (symbol (lib_id "Mechanical:MountingHole") (at 148.59 109.22 0) (unit 1)
+    (in_bom yes) (on_board yes) (fields_autoplaced)
+    (property "Reference" "H27" (id 0) (at 151.13 108.3115 0)
+      (effects (font (size 1.27 1.27)) (justify left))
+    )
+    (property "Value" "MountingHole" (id 1) (at 151.13 111.0866 0)
+      (effects (font (size 1.27 1.27)) (justify left))
+    )
+    (property "Footprint" "MountingHole:MountingHole_3.2mm_M3_ISO14580" (id 2) (at 148.59 109.22 0)
+      (effects (font (size 1.27 1.27)) hide)
+    )
+    (property "Datasheet" "~" (id 3) (at 148.59 109.22 0)
+      (effects (font (size 1.27 1.27)) hide)
+    )
+  )
   (symbol (lib_id "power:GND") (at 90.17 106.045 0) (mirror y) (unit 1)
     (in_bom yes) (on_board yes)
@@
     (pin "6")
     (pin "MP")
+  )
+  (symbol (lib_id "Mechanical:MountingHole") (at 129.54 115.57 0) (unit 1)
+    (in_bom yes) (on_board yes) (fields_autoplaced)
+    (property "Reference" "H26" (id 0) (at 132.08 114.6615 0)
+      (effects (font (size 1.27 1.27)) (justify left))
+    )
+    (property "Value" "MountingHole" (id 1) (at 132.08 117.4366 0)
+      (effects (font (size 1.27 1.27)) (justify left))
+    )
+    (property "Footprint" "MountingHole:MountingHole_3.2mm_M3_ISO14580" (id 2) (at 129.54 115.57 0)
+      (effects (font (size 1.27 1.27)) hide)
+    )
+    (property "Datasheet" "~" (id 3) (at 129.54 115.57 0)
+      (effects (font (size 1.27 1.27)) hide)
+    )
   )
   (symbol (lib_id "power:GND") (at 324.485 47.625 0) (unit 1)
@@
       (reference "H25") (unit 1) (value "MountingHole") (footprint "MountingHole:MountingHole_3.2mm_M3_ISO14580")
     )
+    (path "/b75e22af-d3b0-4241-b996-f4d15f606ce3"
+      (reference "H26") (unit 1) (value "MountingHole") (footprint "MountingHole:MountingHole_3.2mm_M3_ISO14580")
+    )
+    (path "/7ef5b232-f751-4ce1-ac9a-3509e9982f7f"
+      (reference "H27") (unit 1) (value "MountingHole") (footprint "MountingHole:MountingHole_3.2mm_M3_ISO14580")
+    )
     (path "/ba845734-cb29-4a35-9ff6-e58ec1810bec"

Commit message: Andrew Puts a Traffic Cone on Olivia's Happy Highway
Parts:
- added C16: 47uF, Capacitor_SMD:CP_Elec_6.3x7.7, symbol Device:CP1_Small
- U3: symbol Evezor_Library:ESP32-WROOM-32U -> RF_Module:ESP32-WROOM-32U
Connections:
- net GND: now also C16.2
- net VBUS: now also C16.1
Changed lines of the file:
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@@
     (pin "1")
   )
-  (symbol (lib_id "Evezor_Library:ESP32-WROOM-32U") (at 276.86 172.72 0) (unit 1)
+  (symbol (lib_id "RF_Module:ESP32-WROOM-32U") (at 276.86 172.72 0) (unit 1)
     (in_bom yes) (on_board yes)
     (property "Reference" "U3" (id 0) (at 273.05 138.43 0))
     (property "Value" "ESP32-WROOM-32U" (id 1) (at 289.56 138.43 0))
-    (property "Footprint" "RF_Module:ESP32-WROOM-32U_evezor" (id 2) (at 288.29 210.82 0)
-      (effects (font (size 1.27 1.27)) hide)
-    )
-    (property "Datasheet" "https://www.espressif.com/sites/default/files/documentation/esp32-wroom-32d_esp32-wroom-32u_datasheet_en.pdf" (id 3) (at 256.54 171.45 0)
-      (effects (font (size 1.27 1.27)) hide)
+    (property "Footprint" "RF_Module:ESP32-WROOM-32U_evezor" (id 2) (at 284.48 208.28 0)
+      (effects (font (size 1.27 1.27)) hide)
+    )
+    (property "Datasheet" "https://www.espressif.com/sites/default/files/documentation/esp32-wroom-32d_esp32-wroom-32u_datasheet_en.pdf" (id 3) (at 283.21 204.47 0)
+      (effects (font (size 0.38 0.38)) hide)
     )
     (pin "1")
@@
     (pin "1")
   )
+  (symbol (lib_id "Device:CP1_Small") (at 101.6 44.45 0) (unit 1)
+    (in_bom yes) (on_board yes)
+    (property "Reference" "C16" (id 0) (at 103.9114 43.2816 0)
+      (effects (font (size 1.27 1.27)) (justify left))
+    )
+    (property "Value" "47uF" (id 1) (at 103.9114 45.593 0)
+      (effects (font (size 1.27 1.27)) (justify left))
+    )
+    (property "Footprint" "Capacitor_SMD:CP_Elec_6.3x7.7" (id 2) (at 101.6 44.45 0)
+      (effects (font (size 1.27 1.27)) hide)
+    )
+    (property "Datasheet" "~" (id 3) (at 101.6 44.45 0)
+      (effects (font (size 1.27 1.27)) hide)
+    )
+    (pin "1")
+    (pin "2")
+  )
   (symbol (lib_id "LED:SK6812MINI") (at 162.56 229.87 0) (unit 1)
     (in_bom yes) (on_board yes)
@@
       (reference "C15") (unit 1) (value "22uF") (footprint "Capacitor_SMD:C_0805_2012Metric")
     )
+    (path "/15146124-2d10-476a-a8e2-45a0553c4301"
+      (reference "C16") (unit 1) (value "47uF") (footprint "Capacitor_SMD:CP_Elec_6.3x7.7")
+    )
     (path "/51cfa156-df4f-4057-846a-65952de878ca"

Commit message: Sleepy Olivia Draws Lines
Other:
- moved on the sheet: H1, H10, H11, H12, H13, H14, H15, H16, H17, H18, H19, H2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

Commit message: More awake Olivia fixes some things
Parts:
- removed C16: 47uF, Capacitor_SMD:CP_Elec_6.3x7.7, symbol Device:CP1_Small
Other:
- moved on the sheet: C17, H24
Changed lines of the file:
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@@
   (junction (at 135.89 215.9) (diameter 1.016) (color 0 0 0 0)
   )
-  (junction (at 101.6 51.435) (diameter 0) (color 0 0 0 0)
-  )
   (junction (at 278.13 77.47) (diameter 1.016) (color 0 0 0 0)
   )
@@
   (junction (at 394.97 50.8) (diameter 1.016) (color 0 0 0 0)
   )
-  (junction (at 101.6 38.1) (diameter 0) (color 0 0 0 0)
-  )
   (junction (at 405.13 144.78) (diameter 1.016) (color 0 0 0 0)
   )
@@
     (stroke (width 0) (type solid) (color 0 0 0 0))
   )
+  (wire (pts (xy 100.33 51.435) (xy 111.76 51.435))
+    (stroke (width 0) (type solid) (color 0 0 0 0))
+  )
   (wire (pts (xy 309.88 59.69) (xy 309.88 65.405))
     (stroke (width 0) (type solid) (color 0 0 0 0))
@@
     (stroke (width 0) (type solid) (color 0 0 0 0))
   )
+  (wire (pts (xy 100.33 38.1) (xy 111.76 38.1))
+    (stroke (width 0) (type solid) (color 0 0 0 0))
+  )
   (wire (pts (xy 86.36 215.9) (xy 86.36 222.25))
     (stroke (width 0) (type solid) (color 0 0 0 0))
@@
     (stroke (width 0) (type solid) (color 0 0 0 0))
   )
-  (wire (pts (xy 101.6 51.435) (xy 101.6 46.99))
-    (stroke (width 0) (type solid) (color 0 0 0 0))
-  )
   (polyline (pts (xy 217.17 19.05) (xy 416.56 19.05))
     (stroke (width 0) (type dash) (color 0 0 0 0))
@@
     (stroke (width 0) (type solid) (color 0 0 0 0))
   )
-  (wire (pts (xy 90.17 38.1) (xy 90.17 41.91))
+  (wire (pts (xy 100.33 38.1) (xy 100.33 41.91))
     (stroke (width 0) (type solid) (color 0 0 0 0))
   )
@@
     (stroke (width 0) (type solid) (color 0 0 0 0))
   )
-  (wire (pts (xy 101.6 38.1) (xy 101.6 41.91))
-    (stroke (width 0) (type solid) (color 0 0 0 0))
-  )
   (wire (pts (xy 287.02 59.69) (xy 288.925 59.69))
     (stroke (width 0) (type solid) (color 0 0 0 0))
@@
     (stroke (width 0) (type default) (color 0 0 0 0))
   )
-  (wire (pts (xy 90.17 51.435) (xy 101.6 51.435))
-    (stroke (width 0) (type solid) (color 0 0 0 0))
-  )
   (wire (pts (xy 281.94 129.54) (xy 299.72 129.54))
     (stroke (width 0) (type solid) (color 0 0 0 0))
@@
     (stroke (width 0) (type dash) (color 0 0 0 0))
   )
-  (wire (pts (xy 101.6 51.435) (xy 111.76 51.435))
-    (stroke (width 0) (type solid) (color 0 0 0 0))
-  )
-  (wire (pts (xy 90.17 38.1) (xy 101.6 38.1))
-    (stroke (width 0) (type solid) (color 0 0 0 0))
-  )
-  (wire (pts (xy 101.6 38.1) (xy 111.76 38.1))
-    (stroke (width 0) (type solid) (color 0 0 0 0))
-  )
   (wire (pts (xy 62.23 87.63) (xy 72.39 87.63))
     (stroke (width 0) (type solid) (color 0 0 0 0))
@@
     (stroke (width 0) (type solid) (color 0 0 0 0))
   )
-  (wire (pts (xy 90.17 51.435) (xy 90.17 46.99))
+  (wire (pts (xy 100.33 46.99) (xy 100.33 51.435))
     (stroke (width 0) (type solid) (color 0 0 0 0))
   )
@@
     (pin "1")
   )
-  (symbol (lib_id "Device:CP1_Small") (at 101.6 44.45 0) (unit 1)
-    (in_bom yes) (on_board yes)
-    (property "Reference" "C16" (id 0) (at 103.9114 43.2816 0)
-      (effects (font (size 1.27 1.27)) (justify left))
-    )
-    (property "Value" "47uF" (id 1) (at 103.9114 45.593 0)
-      (effects (font (size 1.27 1.27)) (justify left))
-    )
-    (property "Footprint" "Capacitor_SMD:CP_Elec_6.3x7.7" (id 2) (at 101.6 44.45 0)
-      (effects (font (size 1.27 1.27)) hide)
-    )
-    (property "Datasheet" "~" (id 3) (at 101.6 44.45 0)
-      (effects (font (size 1.27 1.27)) hide)
-    )
-    (pin "1")
-    (pin "2")
-  )
   (symbol (lib_id "LED:SK6812MINI") (at 162.56 229.87 0) (unit 1)
     (in_bom yes) (on_board yes)
@@
     )
   )
-  (symbol (lib_id "Device:CP_Small") (at 90.17 44.45 0) (unit 1)
+  (symbol (lib_id "Device:CP_Small") (at 100.33 44.45 0) (unit 1)
     (in_bom yes) (on_board yes)
-    (property "Reference" "C17" (id 0) (at 86.36 41.91 0)
+    (property "Reference" "C17" (id 0) (at 96.52 41.91 0)
       (effects (font (size 1.27 1.27)) (justify left))
     )
-    (property "Value" ".1uF 100V" (id 1) (at 92.71 49.53 90)
+    (property "Value" ".1uF 100V" (id 1) (at 102.87 49.53 90)
       (effects (font (size 1.27 1.27)) (justify left))
     )
-    (property "Footprint" "Capacitor_SMD:C_0805_2012Metric" (id 2) (at 90.17 44.45 0)
+    (property "Footprint" "Capacitor_SMD:C_0805_2012Metric" (id 2) (at 100.33 44.45 0)
       (effects (font (size 1.27 1.27)) hide)
     )
-    (property "Datasheet" "~" (id 3) (at 90.17 44.45 0)
+    (property "Datasheet" "~" (id 3) (at 100.33 44.45 0)
       (effects (font (size 1.27 1.27)) hide)
     )
@@
     (pin "1")
   )
-  (symbol (lib_id "Mechanical:MountingHole") (at 189.865 160.02 0) (unit 1)
+  (symbol (lib_id "Mechanical:MountingHole") (at 187.96 90.17 0) (unit 1)
     (in_bom yes) (on_board yes) (fields_autoplaced)
-    (property "Reference" "H24" (id 0) (at 192.405 159.1115 0)
+    (property "Reference" "H24" (id 0) (at 190.5 89.2615 0)
       (effects (font (size 1.27 1.27)) (justify left))
     )
-    (property "Value" "MountingHole" (id 1) (at 192.405 161.8866 0)
+    (property "Value" "MountingHole" (id 1) (at 190.5 92.0366 0)
       (effects (font (size 1.27 1.27)) (justify left))
     )
-    (property "Footprint" "MountingHole:MountingHole_2.7mm_M2.5_ISO14580" (id 2) (at 189.865 160.02 0)
+    (property "Footprint" "MountingHole:MountingHole_2.7mm_M2.5_ISO14580" (id 2) (at 187.96 90.17 0)
       (effects (font (size 1.27 1.27)) hide)
     )
-    (property "Datasheet" "~" (id 3) (at 189.865 160.02 0)
+    (property "Datasheet" "~" (id 3) (at 187.96 90.17 0)
       (effects (font (size 1.27 1.27)) hide)
     )
@@
       (reference "C15") (unit 1) (value "22uF") (footprint "Capacitor_SMD:C_0805_2012Metric")
     )
-    (path "/15146124-2d10-476a-a8e2-45a0553c4301"
-      (reference "C16") (unit 1) (value "47uF") (footprint "Capacitor_SMD:CP_Elec_6.3x7.7")
-    )
     (path "/51cfa156-df4f-4057-846a-65952de878ca"
