File: cad/line_follower/line_follower/line_follower.kicad_pcb (KiCad board)
At the start: 2 copper layers, 50 x 22 mm, 7 parts, among them J2 Conn_01x03, J5 Conn_01x03, J7 Conn_01x03, J8 Conn_01x03, J9 Conn_01x06_MountingPin

Commit message: Mega monster huge scary big board 4.0 big scary there's like 4 pieces but its actually not that scary huge hugh mungus big board also mousey bites
Parts:
- removed J2, J5, J7, J8: Conn_01x03, Connector_JST:JST_PH_B3B-PH-SM4-TB_1x03-1MP_P2.00mm_Vertical
- added R10: 10K, Resistor_SMD:R_0603_1608Metric, F.Cu at (156.4, 81.3)
- added R12: R100, Resistor_SMD:R_0603_1608Metric, F.Cu at (145.1, 83.5)
- added R13: 10K, Resistor_SMD:R_0603_1608Metric, F.Cu at (145.1, 81.5)
- added R3: R100, Resistor_SMD:R_0603_1608Metric, F.Cu at (175.0, 83.5)
- added R5: 10K, Resistor_SMD:R_0603_1608Metric, F.Cu at (175.0, 81.4)
- added R6: R100, Resistor_SMD:R_0603_1608Metric, F.Cu at (185.1, 83.1)
- added R8: 10K, Resistor_SMD:R_0603_1608Metric, F.Cu at (185.1, 81.3)
- added R9: R100, Resistor_SMD:R_0603_1608Metric, F.Cu at (156.4, 83.5)
- added U1: QRE1113GR, OptoDevice:OnSemi_CASE100CY, F.Cu at (171.7, 88.0)
- added U2: QRE1113GR, OptoDevice:OnSemi_CASE100CY, F.Cu at (185.0, 88.0)
- added U3: QRE1113GR, OptoDevice:OnSemi_CASE100CY, F.Cu at (158.3, 88.0)
- added U4: QRE1113GR, OptoDevice:OnSemi_CASE100CY, F.Cu at (145.0, 88.0)
- moved J9 20.7 mm to (165.6, 76.7), turned to 180 degrees
Connections:
- J9 pad 1: /A -> /Button D
- J9 pad 2: /B -> /Button C
- J9 pad 3: /C -> /Button B
- J9 pad 4: /D -> /Button A
Routing:
- net /A: track 41.0 -> 0.00 mm
- net /Button A: track 0.00 -> 38.8 mm
- net /Button D: track 0.00 -> 30.4 mm
- net /B: track 28.2 -> 0.00 mm
- net /Button C: track 0.00 -> 21.8 mm
- net /Button B: track 0.00 -> 20.3 mm
- net /C: track 18.7 -> 0.00 mm
- net +3V3: track 37.1 -> 54.0 mm, vias 0 -> 4
- net Net-(R3-Pad2): track 0.00 -> 9.94 mm
- net /D: track 8.98 -> 0.00 mm
- net Net-(R6-Pad2): track 0.00 -> 3.63 mm
- net Net-(R12-Pad2): track 0.00 -> 3.24 mm
- net Net-(R9-Pad2): track 0.00 -> 2.62 mm
- net GND: track 0.00 -> 2.03 mm, vias 32 -> 1
Other:
- board text added: "Button"
- board text removed: "Ports"
- board text removed: "S"

Commit message: tracey thingies
Parts:
- moved R12 1.07 mm to (144.1, 83.1), turned to -90 degrees
- moved R13 1.03 mm to (144.9, 80.5)
Routing:
- net +3V3: track 54.0 -> 44.8 mm
- net /Button A: track 38.8 -> 42.7 mm
- net GND: track 2.03 -> 0.00 mm, vias 1 -> 88
- net /Button D: track 30.4 -> 32.1 mm
- net Net-(R12-Pad2): track 3.24 -> 2.08 mm
- net Net-(R3-Pad2): track 9.94 -> 11.0 mm
- net /Button C: track 21.8 -> 22.6 mm
- net Net-(R6-Pad2): track 3.63 -> 4.29 mm
Other:
- board text removed: "Button"

Commit message: Big Kahuna finished, winrar zippy files are funny
Routing:
- net +3V3: track 44.8 -> 53.6 mm
- net GND: vias 88 -> 90
Changed lines of the file:
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@@
       (net 2 "+3V3") (pinfunction "Pin_5") (pintype "passive"))
     (pad "6" smd rect locked (at 2.5 -1.8 180) (size 0.61 2) (layers "F.Cu" "F.Paste" "F.Mask")
-      (net 1 "GND") (pinfunction "Pin_6") (pintype "passive"))
+      (net 1 "GND") (pinfunction "Pin_6") (pintype "passive") (zone_connect 2))
     (pad "MP" smd rect locked (at -5.49 1 180) (size 2.68 3.6) (layers "F.Cu" "F.Paste" "F.Mask")
       (net 1 "GND") (pinfunction "MountPin") (pintype "passive"))
@@
   (via (at 152.5 87.5) (size 0.8) (drill 0.4) (layers "F.Cu" "B.Cu") (free) (net 1))
   (via (at 172.5 87.6) (size 0.8) (drill 0.4) (layers "F.Cu" "B.Cu") (free) (net 1))
+  (via (at 161.99 78.95) (size 0.8) (drill 0.4) (layers "F.Cu" "B.Cu") (free) (net 1))
   (via (at 142.5 72.5) (size 0.8) (drill 0.4) (layers "F.Cu" "B.Cu") (free) (net 1))
   (via (at 157 88.05) (size 0.8) (drill 0.4) (layers "F.Cu" "B.Cu") (free) (net 1))
@@
   (via (at 174.2 86.4) (size 0.8) (drill 0.4) (layers "F.Cu" "B.Cu") (free) (net 1))
   (via (at 150 87.5) (size 0.8) (drill 0.4) (layers "F.Cu" "B.Cu") (free) (net 1))
+  (via (at 163.49 76.43) (size 0.8) (drill 0.4) (layers "F.Cu" "B.Cu") (free) (net 1))
   (via (at 142.45 90.1) (size 0.8) (drill 0.4) (layers "F.Cu" "B.Cu") (free) (net 1))
   (via (at 185 72.5) (size 0.8) (drill 0.4) (layers "F.Cu" "B.Cu") (free) (net 1))
   (via (at 187.5 80) (size 0.8) (drill 0.4) (layers "F.Cu" "B.Cu") (free) (net 1))
   (via (at 171.1 72.6) (size 0.8) (drill 0.4) (layers "F.Cu" "B.Cu") (free) (net 1))
-  (via (at 159.8 83.7) (size 0.8) (drill 0.4) (layers "F.Cu" "B.Cu") (free) (net 1))
+  (via (at 159.58 83.99) (size 0.8) (drill 0.4) (layers "F.Cu" "B.Cu") (free) (net 1))
   (via (at 165 85) (size 0.8) (drill 0.4) (layers "F.Cu" "B.Cu") (free) (net 1))
   (via (at 162.5 85) (size 0.8) (drill 0.4) (layers "F.Cu" "B.Cu") (free) (net 1))
   (via (at 145 75) (size 0.8) (drill 0.4) (layers "F.Cu" "B.Cu") (free) (net 1))
-  (via (at 147.9 86.35) (size 0.8) (drill 0.4) (layers "F.Cu" "B.Cu") (free) (net 1))
+  (via (at 153.93 83.4) (size 0.8) (drill 0.4) (layers "F.Cu" "B.Cu") (free) (net 1))
   (via (at 155.94 77.34) (size 0.8) (drill 0.4) (layers "F.Cu" "B.Cu") (free) (net 1))
   (via (at 150 85) (size 0.8) (drill 0.4) (layers "F.Cu" "B.Cu") (free) (net 1))
@@
   (via (at 154.77 85.52) (size 0.8) (drill 0.4) (layers "F.Cu" "B.Cu") (free) (net 1))
   (via (at 188.21 91.2) (size 0.8) (drill 0.4) (layers "F.Cu" "B.Cu") (free) (net 1))
-  (via (at 177.5 87.5) (size 0.8) (drill 0.4) (layers "F.Cu" "B.Cu") (free) (net 1))
+  (via (at 177.53 88.14) (size 0.8) (drill 0.4) (layers "F.Cu" "B.Cu") (free) (net 1))
   (via (at 187.1 86.05) (size 0.8) (drill 0.4) (layers "F.Cu" "B.Cu") (free) (net 1))
   (via (at 141.99 80.14) (size 0.8) (drill 0.4) (layers "F.Cu" "B.Cu") (free) (net 1))
@@
   (via (at 155 87.5) (size 0.8) (drill 0.4) (layers "F.Cu" "B.Cu") (free) (net 1))
   (via (at 167.5 87.5) (size 0.8) (drill 0.4) (layers "F.Cu" "B.Cu") (free) (net 1))
-  (via (at 155.85 79.7) (size 0.8) (drill 0.4) (layers "F.Cu" "B.Cu") (free) (net 1))
+  (via (at 155.88 78.97) (size 0.8) (drill 0.4) (layers "F.Cu" "B.Cu") (free) (net 1))
   (via (at 177.5 90) (size 0.8) (drill 0.4) (layers "F.Cu" "B.Cu") (free) (net 1))
   (via (at 144.3 92) (size 0.8) (drill 0.4) (layers "F.Cu" "B.Cu") (free) (net 1))
@@
   (via (at 142.5 77.5) (size 0.8) (drill 0.4) (layers "F.Cu" "B.Cu") (free) (net 1))
   (via (at 178.12 91.3) (size 0.8) (drill 0.4) (layers "F.Cu" "B.Cu") (free) (net 1))
-  (via (at 161.05 85.95) (size 0.8) (drill 0.4) (layers "F.Cu" "B.Cu") (free) (net 1))
+  (via (at 159.33 82.63) (size 0.8) (drill 0.4) (layers "F.Cu" "B.Cu") (free) (net 1))
   (via (at 187.5 72.5) (size 0.8) (drill 0.4) (layers "F.Cu" "B.Cu") (free) (net 1))
-  (segment (start 144.245 80.45) (end 144.26 80.465) (width 0.25) (layer "F.Cu") (net 2))
   (segment (start 155.58 81.3) (end 155.58 83.45) (width 0.25) (layer "F.Cu") (net 2))
   (segment (start 174.17 83.47) (end 174.17 84.1) (width 0.25) (layer "F.Cu") (net 2))
   (segment (start 184.25 83.115) (end 184.255 83.12) (width 0.25) (layer "F.Cu") (net 2))
   (segment (start 165.89 81.4) (end 174.16 81.4) (width 0.25) (layer "F.Cu") (net 2))
-  (segment (start 164.072 80.502) (end 164.072 78.486) (width 0.25) (layer "F.Cu") (net 2))
+  (segment (start 164.072 80.408) (end 164.072 78.486) (width 0.25) (layer "F.Cu") (net 2))
   (segment (start 144.1 80.475) (end 144.1 82.275) (width 0.25) (layer "F.Cu") (net 2))
   (segment (start 174.16 81.4) (end 174.17 81.41) (width 0.25) (layer "F.Cu") (net 2))
-  (segment (start 144.075 80.45) (end 144.245 80.45) (width 0.25) (layer "F.Cu") (net 2))
   (segment (start 174.17 83.47) (end 174.17 81.41) (width 0.25) (layer "F.Cu") (net 2))
   (segment (start 184.25 81.3) (end 184.25 83.115) (width 0.25) (layer "F.Cu") (net 2))
   (segment (start 144.1 82.275) (end 144.175 82.2) (width 0.25) (layer "F.Cu") (net 2))
-  (segment (start 164.09 80.52) (end 164.072 80.502) (width 0.25) (layer "F.Cu") (net 2))
   (segment (start 174.17 84.1) (end 174.97 84.9) (width 0.25) (layer "F.Cu") (net 2))
   (segment (start 154.25 81.3) (end 155.58 81.3) (width 0.25) (layer "F.Cu") (net 2))
   (segment (start 165.87 81.42) (end 165.89 81.4) (width 0.25) (layer "F.Cu") (net 2))
+  (segment (start 164.06 80.42) (end 163.99 80.49) (width 0.25) (layer "F.Cu") (net 2))
   (segment (start 183.3 84.9) (end 184.255 83.945) (width 0.25) (layer "F.Cu") (net 2))
   (segment (start 184.255 83.945) (end 184.255 83.12) (width 0.25) (layer "F.Cu") (net 2))
+  (segment (start 156.01 80.49) (end 155.58 80.92) (width 0.25) (layer "F.Cu") (net 2))
+  (segment (start 164.06 80.42) (end 164.072 80.408) (width 0.25) (layer "F.Cu") (net 2))
   (segment (start 153.35 82.2) (end 154.25 81.3) (width 0.25) (layer "F.Cu") (net 2))
   (segment (start 155.58 83.45) (end 155.56 83.47) (width 0.25) (layer "F.Cu") (net 2))
   (segment (start 144.075 80.45) (end 144.1 80.475) (width 0.25) (layer "F.Cu") (net 2))
+  (segment (start 155.58 80.92) (end 155.58 81.3) (width 0.25) (layer "F.Cu") (net 2))
+  (segment (start 163.99 80.49) (end 156.01 80.49) (width 0.25) (layer "F.Cu") (net 2))
   (segment (start 178.85 84.9) (end 183.3 84.9) (width 0.25) (layer "F.Cu") (net 2))
   (segment (start 144.175 82.2) (end 153.35 82.2) (width 0.25) (layer "F.Cu") (net 2))
@@
   (via (at 178.85 84.9) (size 0.8) (drill 0.4) (layers "F.Cu" "B.Cu") (net 2))
   (via (at 174.97 84.9) (size 0.8) (drill 0.4) (layers "F.Cu" "B.Cu") (net 2))
-  (via (at 164.09 80.52) (size 0.8) (drill 0.4) (layers "F.Cu" "B.Cu") (net 2))
-  (segment (start 164.09 80.55) (end 164.09 80.52) (width 0.25) (layer "B.Cu") (net 2))
+  (via (at 164.06 80.42) (size 0.8) (drill 0.4) (layers "F.Cu" "B.Cu") (net 2))
+  (segment (start 164.06 80.42) (end 164.06 80.52) (width 0.25) (layer "B.Cu") (net 2))
   (segment (start 178.85 84.9) (end 174.97 84.9) (width 0.25) (layer "B.Cu") (net 2))
-  (segment (start 165.87 81.42) (end 164.96 81.42) (width 0.25) (layer "B.Cu") (net 2))
-  (segment (start 164.96 81.42) (end 164.09 80.55) (width 0.25) (layer "B.Cu") (net 2))
+  (segment (start 164.06 80.52) (end 164.96 81.42) (width 0.25) (layer "B.Cu") (net 2))
+  (segment (start 164.96 81.42) (end 165.87 81.42) (width 0.25) (layer "B.Cu") (net 2))
   (segment (start 170.766666 87.586666) (end 170.766666 86) (width 0.25) (layer "F.Cu") (net 3))
   (segment (start 171.53 88.35) (end 170.766666 87.586666) (width 0.25) (layer "F.Cu") (net 3))
