File: Big Kahuna Board.kicad_pcb (KiCad board)
At the start: 2 copper layers, 50 x 94 mm, 26 parts, among them J9 Conn_01x06_MountingPin, SW1 SW_Push, SW2 SW_Push, SW3 SW_Push, SW4 SW_Push

Commit message: Big Kahuna finished, winrar zippy files are funny
Parts:
- removed the H1 at (143.9, 44.3)
- removed the H2 at (113.9, 44.3)
- removed the J9 at (148.3, 54.7)
- removed the R4 at (112.9, 50.5)
- added C1: 220uF, Capacitor_SMD:CP_Elec_8x6.5, F.Cu at (123.1, 117.3)
- added D1: led_g, LED_SMD:LED_0603_1608Metric, F.Cu at (113.7, 132.5)
- added D2: SX35_SCHOTTKY, Diode_SMD:D_SMA, F.Cu at (107.1, 116.5)
- added D3: led_g, LED_SMD:LED_0603_1608Metric, F.Cu at (121.6, 132.5)
- added D4: SX35_SCHOTTKY, Diode_SMD:D_SMA, F.Cu at (120.4, 123.6)
- added H1: MountingHole, MountingHole:MountingHole_3.2mm_M3_ISO14580, F.Cu at (143.9, 116.3)
- added H1: MountingHole, MountingHole:MountingHole_3.2mm_M3_ISO14580, F.Cu at (113.9, 106.2)
- added H1: MountingHole, MountingHole:MountingHole_3.2mm_M3_ISO14580, F.Cu at (143.8, 44.3)
- added H1: MountingHole, MountingHole:MountingHole_3.2mm_M3_ISO14580, F.Cu at (143.8, 68.3)
- added H2: MountingHole, MountingHole:MountingHole_3.2mm_M3_ISO14580, F.Cu at (113.8, 68.3)
- added H2: MountingHole, MountingHole:MountingHole_3.2mm_M3_ISO14580, F.Cu at (143.9, 106.2)
- added H2: MountingHole, MountingHole:MountingHole_3.2mm_M3_ISO14580, F.Cu at (113.8, 44.3)
- added H2: MountingHole, MountingHole:MountingHole_3.2mm_M3_ISO14580, F.Cu at (113.9, 116.3)
- added J1: Conn_01x02, Connector_JST:JST_XH_2_VERTICAL, F.Cu at (106.1, 127.4)
- added J2: Conn_01x02, Connector_JST:JST_XH_2_VERTICAL, F.Cu at (129.6, 127.7)
- added J2: Conn_01x03, Connector_JST:JST_PH_B3B-PH-SM4-TB_1x03-1MP_P2.00mm_Vertical, F.Cu at (148.4, 96.2)
- added J4: Servo Header x2, Connector_PinHeader_2.54mm:PinHeader_2x03_P2.54mm_Vertical_SMD, F.Cu at (137.8, 129.3)
- added J5: Conn_01x03, Connector_JST:JST_PH_B3B-PH-SM4-TB_1x03-1MP_P2.00mm_Vertical, F.Cu at (138.9, 96.2)
- added J6: Conn_01x02, Connector_JST:JST_XH_2_VERTICAL, F.Cu at (138.7, 117.7)
- added J7: Conn_01x03, Connector_JST:JST_PH_B3B-PH-SM4-TB_1x03-1MP_P2.00mm_Vertical, F.Cu at (129.4, 96.2)
- added J8: Conn_01x03, Connector_JST:JST_PH_B3B-PH-SM4-TB_1x03-1MP_P2.00mm_Vertical, F.Cu at (119.9, 96.2)
- added J9: Conn_01x06_MountingPin, Connector_FFC-FPC:TE_84952-6_1x06-1MP_P1.0mm_Horizontal, F.Cu at (148.3, 126.6)
- added J9: Conn_01x06_MountingPin, Connector_FFC-FPC:TE_84952-6_1x06-1MP_P1.0mm_Horizontal, F.Cu at (129.4, 69.9)
- added J9: Conn_01x06_MountingPin, Connector_FFC-FPC:TE_84952-6_1x06-1MP_P1.0mm_Horizontal, F.Cu at (148.2, 54.6)
- added J9: Conn_01x06_MountingPin, Connector_FFC-FPC:TE_84952-6_1x06-1MP_P1.0mm_Horizontal, F.Cu at (109.5, 95.9)
- added Q1: LOW PWR FET, Package_TO_SOT_SMD:SOT-23, F.Cu at (113.5, 121.5)
- added Q2: LOW PWR FET, Package_TO_SOT_SMD:SOT-23, F.Cu at (119.0, 128.0)
- added R1: 10k, Resistor_SMD:R_0603_1608Metric, F.Cu at (116.3, 131.7)
- added R10: 10K, Resistor_SMD:R_0603_1608Metric, F.Cu at (120.3, 74.6)
- added R12: R100, Resistor_SMD:R_0603_1608Metric, F.Cu at (108.0, 76.4)
- added R13: 10K, Resistor_SMD:R_0603_1608Metric, F.Cu at (108.8, 73.7)
- added R2: 10k, Resistor_SMD:R_0603_1608Metric, F.Cu at (149.4, 116.5)
- added R3: R100, Resistor_SMD:R_0603_1608Metric, F.Cu at (138.8, 76.7)
- added R3: 10k, Resistor_SMD:R_0603_1608Metric, F.Cu at (119.1, 131.7)
- added R4: 10k, Resistor_SMD:R_0603_1608Metric, F.Cu at (149.5, 114.2)
- added R4: 10k, Resistor_SMD:R_0603_1608Metric, F.Cu at (112.8, 50.5)
- added R5: 10K, Resistor_SMD:R_0603_1608Metric, F.Cu at (138.8, 74.7)
- added R6: R100, Resistor_SMD:R_0603_1608Metric, F.Cu at (148.9, 76.4)
- added R8: 10K, Resistor_SMD:R_0603_1608Metric, F.Cu at (148.9, 74.6)
- added R9: R100, Resistor_SMD:R_0603_1608Metric, F.Cu at (120.2, 76.7)
- added REF**: r, MountingHole:drilled_0_3, F.Cu at (112.0, 87.3)
- added REF**: r, MountingHole:drilled_0_3, F.Cu at (113.0, 111.3)
- added REF**: r, MountingHole:drilled_0_3, F.Cu at (146.0, 87.3)
- added REF**: r, MountingHole:drilled_0_3, F.Cu at (128.0, 111.3)
- added REF**: r, MountingHole:drilled_0_3, F.Cu at (148.0, 87.3)
- added REF**: r, MountingHole:drilled_0_3, F.Cu at (144.7, 111.3)
- added REF**: r, MountingHole:drilled_0_3, F.Cu at (110.0, 111.3)
- added REF**: r, MountingHole:drilled_0_3, F.Cu at (146.0, 111.3)
- added REF**: r, MountingHole:drilled_0_3, F.Cu at (108.8, 87.3)
- added REF**: r, MountingHole:drilled_0_3, F.Cu at (110.0, 87.3)
- added REF**: r, MountingHole:drilled_0_3, F.Cu at (131.0, 111.3)
- added REF**: r, MountingHole:drilled_0_3, F.Cu at (130.0, 87.3)
- added REF**: r, MountingHole:drilled_0_3, F.Cu at (126.7, 111.3)
- added REF**: r, MountingHole:drilled_0_3, F.Cu at (129.0, 111.3)
- added REF**: r, MountingHole:drilled_0_3, F.Cu at (113.0, 87.3)
- added REF**: r, MountingHole:drilled_0_3, F.Cu at (130.0, 111.3)
- added REF**: r, MountingHole:drilled_0_3, F.Cu at (129.0, 87.3)
- added REF**: r, MountingHole:drilled_0_3, F.Cu at (128.0, 87.3)
- added REF**: r, MountingHole:drilled_0_3, F.Cu at (126.8, 87.3)
- added REF**: r, MountingHole:drilled_0_3, F.Cu at (131.0, 87.3)
- added REF**: r, MountingHole:drilled_0_3, F.Cu at (147.0, 111.3)
- added REF**: r, MountingHole:drilled_0_3, F.Cu at (111.0, 87.3)
- added REF**: r, MountingHole:drilled_0_3, F.Cu at (108.7, 111.3)
- added REF**: r, MountingHole:drilled_0_3, F.Cu at (149.0, 87.3)
- added REF**: r, MountingHole:drilled_0_3, F.Cu at (149.0, 111.3)
- added REF**: r, MountingHole:drilled_0_3, F.Cu at (147.0, 87.3)
- added REF**: r, MountingHole:drilled_0_3, F.Cu at (111.0, 111.3)
- added REF**: r, MountingHole:drilled_0_3, F.Cu at (112.0, 111.3)
- added REF**: r, MountingHole:drilled_0_3, F.Cu at (144.8, 87.3)
- added REF**: r, MountingHole:drilled_0_3, F.Cu at (148.0, 111.3)
- added U1: QRE1113GR, OptoDevice:OnSemi_CASE100CY, F.Cu at (135.5, 81.3)
- added U2: QRE1113GR, OptoDevice:OnSemi_CASE100CY, F.Cu at (148.8, 81.3)
- added U3: QRE1113GR, OptoDevice:OnSemi_CASE100CY, F.Cu at (122.2, 81.3)
- added U4: QRE1113GR, OptoDevice:OnSemi_CASE100CY, F.Cu at (108.8, 81.3)
Routing:
- net +3V3: track 35.0 -> 125.8 mm, vias 0 -> 4
- net +VDC: track 0.00 -> 71.0 mm
- net /Thing 1: track 0.00 -> 60.4 mm, vias 0 -> 4
- net /Thing 2: track 0.00 -> 53.6 mm, vias 0 -> 2
- net /Button A: track 39.5 -> 82.2 mm
- net /A: track 0.00 -> 41.0 mm
- net /Button D: track 10.9 -> 43.0 mm
- net /B: track 0.00 -> 28.2 mm
- net /Button C: track 20.8 -> 43.4 mm
- net /Button B: track 30.1 -> 50.5 mm
- net /C: track 0.00 -> 18.7 mm
- net Net-(D2-Pad2): track 0.00 -> 16.3 mm
- net /SERVO_2: track 0.00 -> 13.2 mm
- net Net-(R3-Pad2): track 0.00 -> 11.0 mm
- net Net-(D4-Pad2): track 0.00 -> 10.2 mm
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Other:
- board text added: "+"
- board text added: "Ports"
- board text added: "S"
- board text added: "Servo/Mosfet Board"
