File: cad/button/line_follower/line_follower.kicad_pcb (KiCad board)
At the start: 2 copper layers, 50 x 22 mm, 33 parts, among them J2 Conn_01x03, J5 Conn_01x03, J7 Conn_01x03, J8 Conn_01x03, J9 Conn_01x06_MountingPin, Q1 LOW PWR FET, SW1 SW_Push, SW2 SW_Push, SW3 SW_Push, SW4 SW_Push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

Commit message: Big Kahuna finished, winrar zippy files are funny
Parts:
- removed C1: 220uF, Capacitor_SMD:CP_Elec_10x12.5
- removed D1: led_g, LED_SMD:LED_0603_1608Metric
- removed D2: SX35_SCHOTTKY, Diode_SMD:D_SMA
- removed J2, J5, J7, J8: Conn_01x03, Connector_JST:JST_PH_B3B-PH-SM4-TB_1x03-1MP_P2.00mm_Vertical
- removed Q1: LOW PWR FET, Package_TO_SOT_SMD:SOT-23
- removed R1, R2: 10k, Resistor_SMD:R_0603_1608Metric
- removed R10, R13, R5, R8: 10K, Resistor_SMD:R_0603_1608Metric
- removed R12, R3, R6, R9: R100, Resistor_SMD:R_0603_1608Metric
- removed U1, U2, U3, U4: QRE1113GR, OptoDevice:OnSemi_CASE100CY
