File: cad/button/line_follower/line_follower.kicad_sch (KiCad schematic)
At the start: 37 parts, among them J1 Conn_01x02, J2 Conn_01x03, J3 Conn_01x02, J4 Servo Header x2, J5 Conn_01x03, J6 Conn_01x02, J7 Conn_01x03, J8 Conn_01x03, J9 Conn_01x06_MountingPin, Q1 LOW PWR FET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

Commit message: Big Kahuna finished, winrar zippy files are funny
Parts:
- removed C1: 220uF, Capacitor_SMD:CP_Elec_10x12.5, symbol Device:CP_Small
- removed D1: led_g, LED_SMD:LED_0603_1608Metric, symbol Device:LED
- removed D2: SX35_SCHOTTKY, Diode_SMD:D_SMA, symbol Device:D_Schottky
- removed J1, J3, J6: Conn_01x02, Evezor_extras:CONN_JST_XH_2_VERTICAL, symbol Connector_Generic_MountingPin:Conn_01x02_MountingPin
- removed J2, J5, J7, J8: Conn_01x03, Connector_JST:JST_PH_B3B-PH-SM4-TB_1x03-1MP_P2.00mm_Vertical, symbol Connector_Generic_MountingPin:Conn_01x03_MountingPin
- removed J4: Servo Header x2, Evezor_extras:PinHeader_2x03_P2.54mm_Vertical_SMD, symbol Connector_Generic:Conn_02x03_Counter_Clockwise
- removed Q1: LOW PWR FET, Package_TO_SOT_SMD:SOT-23, symbol Device:Q_NMOS_GSD
- removed R1, R2: 10k, Resistor_SMD:R_0603_1608Metric, symbol Device:R_Small
- removed R10, R13, R5, R8: 10K, Resistor_SMD:R_0603_1608Metric, symbol Device:R_Small
- removed R12, R3, R6, R9: R100, Resistor_SMD:R_0603_1608Metric, symbol Device:R_Small
- removed U1, U2, U3, U4: QRE1113GR, OptoDevice:OnSemi_CASE100CY, symbol Sensor_Proximity:QRE1113
