File: cad/servo_board/line_follower/line_follower.kicad_pcb (KiCad board)
At the start: 2 copper layers, 50 x 22 mm, 18 parts, among them J1 Conn_01x02, J2 Conn_01x02, J4 Servo Header x2, J6 Conn_01x02, J9 Conn_01x06_MountingPin, Q1 LOW PWR FET, Q2 LOW PWR FET

Commit message: tracey thingies
Parts:
- moved J6 1.46 mm to (174.8, 76.4)
- moved J2 0.52 mm to (165.7, 86.4)
- moved Q1 0.36 mm to (149.6, 80.3)
- moved J1 0.30 mm to (142.3, 86.2)
- moved J4 0.17 mm to (174.0, 88.0)
- moved C1 0.08 mm to (159.2, 76.0)
Routing:
- net +VDC: track 65.6 -> 71.0 mm
- net /Thing 1: track 57.5 -> 60.4 mm
- net Net-(D2-Pad2): track 14.9 -> 16.3 mm
- net /Thing 2: track 52.5 -> 53.6 mm
- net /SERVO_2: track 12.6 -> 13.2 mm
- net GND: vias 14 -> 86
Other:
- board text removed: "b"
- board text removed: "c"

Commit message: Big Kahuna finished, winrar zippy files are funny
Routing:
- net GND: vias 86 -> 87
Other:
- board text added: "+"
- board text added: "S"
- board text added: "Servo/Mosfet Board"
- board text removed: "Button"
Changed lines of the file:
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@@
     )
   )
-  (gr_rect (start 179 82) (end 181 84) (layer "F.SilkS") (width 0.15) (fill none))
-  (gr_rect (start 179 84) (end 181 86) (layer "F.SilkS") (width 0.15) (fill none))
-  (gr_rect (start 179 88) (end 181 90) (layer "F.SilkS") (width 0.15) (fill none))
-  (gr_rect (start 179 86) (end 181 88) (layer "F.SilkS") (width 0.15) (fill none))
-  (gr_rect (start 179 90) (end 181 92) (layer "F.SilkS") (width 0.15) (fill none))
-  (gr_rect (start 179 80) (end 181 82) (layer "F.SilkS") (width 0.15) (fill none))
+  (gr_rect (start 179.26 81.94) (end 181.26 83.94) (layer "F.SilkS") (width 0.15) (fill none))
+  (gr_rect (start 179.26 83.94) (end 181.26 85.94) (layer "F.SilkS") (width 0.15) (fill none))
+  (gr_rect (start 179.26 87.94) (end 181.26 89.94) (layer "F.SilkS") (width 0.15) (fill none))
+  (gr_rect (start 179.26 85.94) (end 181.26 87.94) (layer "F.SilkS") (width 0.15) (fill none))
+  (gr_rect (start 179.26 89.94) (end 181.26 91.94) (layer "F.SilkS") (width 0.15) (fill none))
+  (gr_rect (start 179.26 79.94) (end 181.26 81.94) (layer "F.SilkS") (width 0.15) (fill none))
   (gr_circle (center 180 75) (end 181.6 75) (layer "Cmts.User") (width 0.4) (fill none))
   (gr_circle (center 150 75) (end 151.6 75) (layer "Cmts.User") (width 0.4) (fill none))
@@
   (gr_arc (start 190 91.31005) (mid 189.505025 92.505025) (end 188.31005 93) (layer "Edge.Cuts") (width 0.4))
   (gr_line (start 190 72.68995) (end 190 91.31005) (layer "Edge.Cuts") (width 0.4))
-  (gr_text "A" (at 180 85 270) (layer "F.SilkS")
+  (gr_text "Servo/Mosfet Board" (at 164.98 81.83) (layer "B.SilkS")
+    (effects (font (size 3 3) (thickness 0.6)) (justify mirror))
+  )
+  (gr_text "+" (at 178.65 88.05) (layer "F.SilkS")
+    (effects (font (size 1 1) (thickness 0.25)))
+  )
+  (gr_text "A" (at 180.26 84.94 270) (layer "F.SilkS")
     (effects (font (size 1 1) (thickness 0.15)))
+  )
+  (gr_text "G" (at 178.69 85.57) (layer "F.SilkS")
+    (effects (font (size 1 1) (thickness 0.25)))
   )
   (gr_text "B" (at 160.528 90.451) (layer "F.SilkS")
     (effects (font (size 2.5 2.5) (thickness 0.5)))
   )
-  (gr_text "Button" (at 165.02 63.02) (layer "F.SilkS")
-    (effects (font (size 2 2) (thickness 0.5)))
+  (gr_text "+" (at 168.64 88.03) (layer "F.SilkS")
+    (effects (font (size 1 1) (thickness 0.25)))
+  )
+  (gr_text "S" (at 168.83 90.63) (layer "F.SilkS")
+    (effects (font (size 1 1) (thickness 0.25)))
+  )
+  (gr_text "G" (at 168.75 85.48) (layer "F.SilkS")
+    (effects (font (size 1 1) (thickness 0.25)))
   )
   (gr_text "A" (at 151.384 87.376) (layer "F.SilkS")
     (effects (font (size 2.5 2.5) (thickness 0.5)))
   )
-  (gr_text "C" (at 168.656 89.916) (layer "F.SilkS")
-    (effects (font (size 2.5 2.5) (thickness 0.5)))
+  (gr_text "C" (at 170.32 83.44) (layer "F.SilkS")
+    (effects (font (size 2 2) (thickness 0.5)))
   )
-  (gr_text "G" (at 180 81 270) (layer "F.SilkS")
+  (gr_text "G" (at 180.26 80.94 270) (layer "F.SilkS")
     (effects (font (size 1 1) (thickness 0.15)))
   )
-  (gr_text "C" (at 180 89 270) (layer "F.SilkS")
+  (gr_text "S" (at 178.65 90.65) (layer "F.SilkS")
+    (effects (font (size 1 1) (thickness 0.25)))
+  )
+  (gr_text "D\n" (at 177.52 83.46) (layer "F.SilkS")
+    (effects (font (size 2 2) (thickness 0.5)))
+  )
+  (gr_text "C" (at 180.26 88.94 270) (layer "F.SilkS")
     (effects (font (size 1 1) (thickness 0.15)))
   )
-  (gr_text "D" (at 180 91 270) (layer "F.SilkS")
+  (gr_text "D" (at 180.26 90.94 270) (layer "F.SilkS")
     (effects (font (size 1 1) (thickness 0.15)))
   )
-  (gr_text "3V" (at 180 83 270) (layer "F.SilkS")
+  (gr_text "3V" (at 180.26 82.94 270) (layer "F.SilkS")
     (effects (font (size 1 1) (thickness 0.15)))
   )
-  (gr_text "B" (at 180 87 270) (layer "F.SilkS")
+  (gr_text "B" (at 180.26 86.94 270) (layer "F.SilkS")
     (effects (font (size 1 1) (thickness 0.15)))
   )
@@
   (via (at 159.36 72.86) (size 0.8) (drill 0.4) (layers "F.Cu" "B.Cu") (free) (net 1))
   (via (at 182.23 81.34) (size 0.8) (drill 0.4) (layers "F.Cu" "B.Cu") (free) (net 1))
-  (via (at 168.59 80.66) (size 0.8) (drill 0.4) (layers "F.Cu" "B.Cu") (free) (net 1))
+  (via (at 168.8 80.49) (size 0.8) (drill 0.4) (layers "F.Cu" "B.Cu") (free) (net 1))
   (via (at 179.85 91.07) (size 0.8) (drill 0.4) (layers "F.Cu" "B.Cu") (free) (net 1))
   (via (at 153.78 89.16) (size 0.8) (drill 0.4) (layers "F.Cu" "B.Cu") (free) (net 1))
   (via (at 141.224 75.184) (size 0.8) (drill 0.4) (layers "F.Cu" "B.Cu") (free) (net 1))
   (via (at 188.37 89.5) (size 0.8) (drill 0.4) (layers "F.Cu" "B.Cu") (free) (net 1))
+  (via (at 186.53 85.42) (size 0.8) (drill 0.4) (layers "F.Cu" "B.Cu") (free) (net 1))
   (via (at 146.83 72.31) (size 0.8) (drill 0.4) (layers "F.Cu" "B.Cu") (free) (net 1))
   (via (at 144.54 79.63) (size 0.8) (drill 0.4) (layers "F.Cu" "B.Cu") (free) (net 1))
